File: Hardware/Earthquake Alarm.kicad_sch (KiCad schematic)
At the start: 15 parts

Commit message: Finished USB based design
Parts:
- added LED1: XL-3030UWC-1W-3V, easyeda2kicad:LED-SMD_L3.0-W3.0_WHITE, symbol easyeda2kicad:XL-3030UWC-1W-3V
- added Q1, Q2: AO3400A, easyeda2kicad:SOT-23-3_L2.9-W1.6-P1.90-LS2.8-BR, symbol easyeda2kicad:AO3400A
- added R1, R2, R3, R4, R5: 33Ω, easyeda2kicad:R0805, symbol easyeda2kicad:33Ω 0805 150V
- added R6, R8: 100Ω 0402 50V, easyeda2kicad:R0402, symbol easyeda2kicad:100Ω 0402 50V
- added R7, R9: 10kΩ 0402 50V, easyeda2kicad:R0402, symbol easyeda2kicad:10kΩ 0402 50V
- gave numbers to parts that had none: 15
Connections:
- net Buzzer: now also R6.1
- net GND: now also Q1.2 (S), Q2.2 (S), R7.1, R9.1
- net LED: now also R8.1
- net +5V: now reaches C6.2, CN1.1 (VCC), U2.2 (Vin)
- net +5V: now also BUZZER1.1, R1.2, R2.2, R3.2, R4.2, R5.2
- net at BUZZER1.2: now also Q1.3 (D)
- new net: Q1.1 (G), R6.2, R7.2
- new net: Q2.1 (G), R8.2, R9.2
- new net: LED1.2 (K), Q2.3 (D)
- new net: LED1.1 (A), R1.1, R2.1, R3.1, R4.1, R5.1
Other:
- moved on the sheet: BUZZER1
